File: stopwatch-point-3.kicad_pcb (KiCad board)
At the start: 4 copper layers, 46 x 40.2 mm, 85 parts, among them J1 lipo, J4 USB_C_Receptacle_USB2.0_16P, J5 LS013B7DH03, Q1 AO3400A, Q2 2N7002, SW10 SW_Push, SW11 SW_Push_SPDT, SW5 BOOT, SW6 RESET, SW7 SW_Push, SW8 SW_Push, SW9 SW_Push, U1 USBLC6-2SC6, U2 TPS63001, U3 MAX17048, U4 BQ24075RGT, U8 STM32U073CBTx, Y1 ABS07-32.768KHZ-T

Commit message: minor fixes to pcb
Parts:
- moved D3 0.22 mm to (131.7, 80.1), turned to 55 degrees
- moved D1 0.19 mm to (146.1, 80.2), turned to -55 degrees
Routing:
- net GND: track 54.2 -> 55.7 mm

Commit message: add art + minor pcb changes
Parts:
- removed C1: 10uF, Capacitor_SMD:C_0402_1005Metric
- added G***: LOGO, LOGO, F.Cu at (139.6, 61.8)
- added G***: LOGO, LOGO, F.Cu at (138.9, 75.5)
- added G***: LOGO, LOGO, B.Cu at (138.1, 61.6)
- TP2: footprint TestPoint:TestPoint_Pad_D2.0mm -> TestPoint:TestPoint_Pad_2.0x2.0mm
- moved C22 1.20 mm to (145.4, 51.5), turned to -45 degrees
- moved C20 0.92 mm to (139.4, 48.4)
- moved TP2 0.27 mm to (153.8, 51.0)
- moved C18 0.14 mm to (143.4, 47.9)
- moved C26 0.14 mm to (144.4, 48.9)
- moved R16 0.10 mm to (139.4, 45.5)
Routing:
- net GND: track 55.7 -> 54.8 mm
- net RESET: track 47.6 -> 47.1 mm

Commit message: pcb + art edits
Changed lines of the file:
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@@
 	)
 	(via
-		(at 152 61)
+		(at 150.06 60.21)
 		(size 0.6)
 		(drill 0.3)
@@
 	)
 	(zone
-		(net 2)
-		(net_name "GND")
-		(layers "F.Cu" "B.Cu")
-		(hatch edge 0.5)
-		(connect_pads yes
-			(clearance 0.2)
-		)
-		(min_thickness 0.25)
-		(filled_areas_thickness no)
-		(fill yes
-			(thermal_gap 0.2)
-			(thermal_bridge_width 0.5)
-		)
-		(polygon
-			(pts
-				(xy 167.33 55.15) (xy 167.34 57.11) (xy 170.13 57.13) (xy 170.12 55.16)
-			)
-		)
-	)
-	(zone

Commit message: minor edits
Parts:
- C10, C28: value 0.1uF -> 100nF
- C13: footprint Capacitor_SMD:C_0603_1608Metric -> Capacitor_SMD:C_0805_2012Metric
- D1: value LED -> green
- D3: value LED -> orange
- R13: value 100R -> 100
- moved R10 0.33 mm to (131.3, 76.3)
- moved C13 0.32 mm to (128.5, 75.0)
Routing:
- net GND: track 54.8 -> 59.8 mm, vias 170 -> 148
- net PUSH4: track 24.4 -> 25.8 mm
- net PUSH3: track 15.2 -> 16.2 mm
- net VIB: track 16.2 -> 17.2 mm
- net +5V: track 144.4 -> 143.6 mm
- net Net-(U8-PA14): track 29.2 -> 29.9 mm
- net PUSH1: vias 2 -> 3
